File: Hw/solderingChallenge.kicad_sch (KiCad schematic)
At the start: 14 parts, among them J2 SWD, SW1 SW_RST, SW2 On, U1 PY32F002AA15M6TU

Commit message: feat(Hw):Update_csv
Parts:
- C1: LCSC# C235731 -> C38141
Changed lines of the file:
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@@
 			)
 		)
-		(property "LCSC#" "C235731"
+		(property "LCSC#" "C38141"
 			(at 17.272 62.738 0)
 			(effects
